Commit message: tested gripper control in gazebo for 3f
- changed which macro is used
- python 2->3
- tweak P gain

File: robotiq_3f_gripper_visualization/cfg/robotiq-3f-gripper_articulated.xacro (robot description, xacro)
@@ -5,6 +5,15 @@
 -->
 <robot name="robotiq-3f-gripper_articulated" xmlns:xacro="http://ros.org/wiki/xacro">
-        <xacro:include filename="$(find robotiq_3f_gripper_visualization)/cfg/robotiq-3f-gripper_articulated_macro.xacro" />
-        <xacro:robotiq-3f-gripper_articulated prefix=""/>
+        <link name="world"/>
+        <xacro:include filename="$(find robotiq_3f_gripper_visualization)/cfg/robotiq_hand_macro.urdf.xacro" />
+        <xacro:robotiq_hand prefix="l_" parent="world">
+                <origin xyz="0 0 0.1" rpy="0 0 0" />
+        </xacro:robotiq_hand>
+        <gazebo>
+                <plugin name="RobotiqHandPlugin" filename="libRobotiqHandPlugin.so">
+                        <side>left</side>
+                        <kp_position>5</kp_position>
+                </plugin>
+        </gazebo>
 <!--
         <xacro:include filename="$(find robotiq_3f_gripper_visualization)/cfg/robotiq-3f-gripper_finger_articulated_macro.xacro" />

File: robotiq_3f_gripper_visualization/cfg/robotiq_hand_macro.urdf.xacro (robot description, xacro)
@@ -632,5 +632,5 @@
     </gazebo>
   </xacro:macro>
-  <xacro:macro name="robotiq_hand" params="prefix *origin reflect parent">
+  <xacro:macro name="robotiq_hand" params="prefix *origin parent">
     <!-- joint attaching parent link to robotiq hand -->
     <joint name="${prefix}robotiq_hand_joint" type="fixed">
