Commit message: grippers no longer close randomly, added springs
unfortunately the gripping motions don't match the real gripper, because
idk how the real grippers work and I don't think it matters

File: robotiq_3f_gripper_visualization/cfg/robotiq_hand_macro.urdf.xacro (robot description, xacro)
@@ -7,712 +7,814 @@
 -->
 <robot xmlns:xacro="http://www.ros.org/wiki/xacro" name="robotiq_hand">
-  <xacro:macro name="robotiq_finger" params="prefix">
-    <!-- Link list -->
-    <!-- Link 0 -->
-    <link name="${prefix}link_0">
-      <visual>
-        <origin xyz="0 0 0" rpy="0 0 0"/>
-        <geometry>
-          <mesh filename="package://robotiq_3f_gripper_visualization/meshes/robotiq-3f-gripper_articulated/visual/link_0.dae" />
-        </geometry>
-        <material name="green">
-          <color rgba="0 1 0 1"/>
-        </material>
-      </visual>
-      <collision>
-        <origin rpy="0 0 0" xyz="0 0 0"/>
-        <geometry>
-          <mesh filename="package://robotiq_3f_gripper_visualization/meshes/robotiq-3f-gripper_articulated/collision/link_0.STL" />
-        </geometry>
-        <material name="yellow">
-          <color rgba="0 1 1 1"/>
-        </material>
-      </collision>
-      <inertial>
-        <mass value="0.1"/>
-        <origin xyz="-0.01 0 0"/>
-        <inertia ixx="0.000018" ixy="0" ixz="0" iyy="0.000025" iyz="0" izz="0.000025"/>
-      </inertial>
-    </link>
-    <gazebo reference="${prefix}link_0">
-      <mu1>1.1</mu1>
-      <mu2>1.1</mu2>
-    </gazebo>
-    <!-- Link 1 -->
-    <link name="${prefix}link_1">
-      <visual>
-        <origin rpy="0 0 ${3.1416/2}" xyz="0 0.05717 0"/>
-        <geometry>
-          <mesh filename="package://robotiq_3f_gripper_visualization/meshes/robotiq-3f-gripper_articulated/visual/link_1.dae" />
-        </geometry>
-        <material name="green"/>
-      </visual>
-      <collision>
-        <origin rpy="0 0 ${3.1416/2}" xyz="0 0.05717 0"/>
-        <geometry>
-          <mesh filename="package://robotiq_3f_gripper_visualization/meshes/robotiq-3f-gripper_articulated/collision/link_1.STL"/>
-        </geometry>
-        <material name="yellow">
-          <color rgba="0 1 1 1"/>
-        </material>
-      </collision>
-      <inertial>
-        <origin rpy="0 0 ${3.1416/2}" xyz="0.00053 0.03218 0"/>
-        <mass value="0.047"/>
-        <inertia ixx= "0.00000499332"
-                 ixy= "0.00000091312"
-                 ixz="-0.00000000120"
-                 iyy= "0.00006434531"
-                 iyz="-0.00000000007"
-                 izz= "0.00006061917"/>
-      </inertial>
-    </link>
-    <gazebo reference="${prefix}link_1">
-      <mu1>1.1</mu1>
-      <mu2>1.1</mu2>
-    </gazebo>
-    <!-- Link 2 -->
-    <link name="${prefix}link_2">
-      <visual>
-        <origin rpy="0 0 ${3.1416/2}" xyz="0 0.03810 0.0075"/>
-        <geometry>
-          <mesh filename="package://robotiq_3f_gripper_visualization/meshes/robotiq-3f-gripper_articulated/visual/link_2.dae" />
-        </geometry>
-        <material name="green"/>
-      </visual>
-      <collision>
-        <origin rpy="0 0 ${3.1416/2}" xyz="0 0.03810 0.0075"/>
-          <geometry>
-            <mesh filename="package://robotiq_3f_gripper_visualization/meshes/robotiq-3f-gripper_articulated/collision/link_2.STL"/>
-          </geometry>
-        <material name="yellow"/>
-      </collision>
-      <inertial>
-        <origin rpy="0 0 ${3.1416/2}" xyz="0.00048 0.02167 0.00018"/>
-        <mass value="0.03284"/>
-        <inertia ixx="0.00000348008"
-                 ixy="0.00000031940"
-                 ixz="0.00000013041"
-                 iyy="0.00002248123"
-                 iyz="0.00000000291"
-                 izz="0.00001986346"/>
-      </inertial>
-    </link>
-    <gazebo reference="${prefix}link_2">
-      <mu1>1.1</mu1>
-      <mu2>1.1</mu2>
-    </gazebo>
-    <!-- Link 3 -->
-    <link name="${prefix}link_3">
-      <visual>
-        <origin xyz="0 0 0" rpy="0 0 0"/>
-        <geometry>
-          <mesh filename="package://robotiq_3f_gripper_visualization/meshes/robotiq-3f-gripper_articulated/visual/link_3.dae" />
-        </geometry>
-        <material name="green"/>
-      </visual>
-      <collision>
-        <origin xyz="0 0 0" rpy="0 0 0"/>
-        <geometry>
-          <mesh filename="package://robotiq_3f_gripper_visualization/meshes/robotiq-3f-gripper_articulated/collision/link_3.STL"/>
-        </geometry>
-        <material name="yellow"/>
-      </collision>
-      <inertial>
-        <origin rpy="0 0 0" xyz="0.01626 0.00049 0.0002"/>
-        <mass value="0.03354"/>
-        <inertia ixx="0.00000305151"
-                 ixy="0.00000089792"
-                 ixz="0.00000000249"
-                 iyy="0.00001427978"
-                 iyz="-0.00000001191"
-                 izz="0.00001264126"/>
-      </inertial>
-    </link>
-    <gazebo reference="${prefix}link_3">
-      <mu1>1.1</mu1>
-      <mu2>1.1</mu2>
-    </gazebo>
-    <!-- Link proximal actuating hinge -->
-    <link name="${prefix}link_proximal_actuating_hinge">
-      <visual>
-        <origin rpy="0 0 0" xyz="0.01429 0 0"/>
-        <geometry>
-          <box size="0.02858 .0075 .002"/>
-        </geometry>
-      </visual>
-      <collision>
-        <origin rpy="0 0 0" xyz="0.01429 0 0"/>
-         <geometry>
-          <box size="0.02858 .0075 .002"/>
-        </geometry>
-      </collision>
-      <inertial>
-        <origin rpy="0 0 0" xyz="0.0012 -0.00162 -0.00161"/>
-        <mass value="0.02647"/>
-        <inertia ixx= "0.00000156447"
-                 ixy= "0.000000236226"
-                 ixz="-0.00000014862"
-                 iyy= "0.00000221068"
-                 iyz="-0.00000014369"
-                 izz= "0.00000323175"/>
-      </inertial>
-    </link>
-    <gazebo reference="${prefix}link_proximal_actuating_hinge">
-      <mu1>1.1</mu1>
-      <mu2>1.1</mu2>
-    </gazebo>
-    <!-- Link paraproximal actuating hinge -->
-    <link name="${prefix}link_paraproximal_actuating_hinge">
-      <visual>
-        <origin rpy="0 0 0" xyz="0.01143 0 0"/>
-        <geometry>
-          <box size="0.02286 .0075 .002"/>
-        </geometry>
-      </visual>
-      <collision>
-        <origin rpy="0 0 0" xyz="0.01143 0 0"/>
-         <geometry>
-          <box size="0.02286 .0075 .002"/>
-        </geometry>
-      </collision>
-      <inertial>
-        <origin rpy="0 0 0" xyz="0.0064 0 0"/>
-        <!-- copied from proximal_actuating_hinge -->
-        <mass value="0.00362"/>
-        <inertia ixx= "0.00000012043"
-                 ixy= "0"
-                 ixz= "0"
-                 iyy= "0.00000053588"
-                 iyz= "0"
-                 izz= "0.00000065322"/>
-      </inertial>
-    </link>
-    <gazebo reference="${prefix}link_paraproximal_actuating_hinge">
-      <mu1>1.1</mu1>
-      <mu2>1.1</mu2>
-    </gazebo>
-    <!-- Link proximal actuating bar -->
-    <link name="${prefix}link_proximal_actuating_bar">
-      <visual>
-        <origin rpy="0 0 0" xyz="0.026789 0 0"/>
-        <geometry>
-          <box size="0.05398 .0075 .002"/>
-        </geometry>
-      </visual>
-      <collision>
-        <origin rpy="0 0 0" xyz="0.026789 0 0"/>
-         <geometry>
-          <box size="0.05398 .0075 .002"/>
-        </geometry>
-      </collision>
-      <inertial>
-        <origin rpy="0 0 0" xyz="0.02699 -0.00122 0"/>
-        <mass value="0.00659"/>
-        <inertia ixx= "0.00000008348"
-                 ixy="-0.0000002179"
-                 ixz= "0.00000000134"
-                 iyy= "0.00000719076"
-                 iyz= "0"
-                 izz= "0.00000718272"/>
-      </inertial>
-    </link>
-    <gazebo reference="${prefix}link_proximal_actuating_bar">
-      <mu1>1.1</mu1>
-      <mu2>1.1</mu2>
-    </gazebo>
-    <!-- Link paraproximal bar -->
-    <link name="${prefix}link_paraproximal_bar">
-      <visual>
-        <origin rpy="0 0 0" xyz="0.02885 0 0"/>
-        <geometry>
-          <box size="0.05770 .0075 .002"/>
-        </geometry>
-      </visual>
-      <collision>
-        <origin rpy="0 0 0" xyz="0.02885 0 0"/>
-         <geometry>
-          <box size="0.05770 .0075 .002"/>
-        </geometry>
-      </collision>
-      <inertial>
-        <origin rpy="0 0 0" xyz="0.02858 -0.00129 0"/>
-        <mass value="0.00732"/>
-        <inertia ixx= "0.00000009065"
-                 ixy="-0.00000027047"
-                 ixz= "0.00000000142"
-                 iyy= "0.00000878034"
-                 iyz= "0"
-                 izz= "0.00000877558"/>
-      </inertial>
-    </link>
-    <gazebo reference="${prefix}link_paraproximal_bar">
-      <mu1>1.1</mu1>
-      <mu2>1.1</mu2>
-    </gazebo>
-    <!-- Link median actuating hinge -->
-    <link name="${prefix}link_median_actuating_hinge">
-      <visual>
-        <origin rpy="0 0 0" xyz="0 0 0"/>
-        <geometry>
-          <box size=".02 .02 .002"/>
-        </geometry>
-      </visual>
-      <collision>
-        <origin rpy="0 0 0" xyz="0 0 0"/>
-         <geometry>
-          <box size=".02 .02 .002"/>
-        </geometry>
-      </collision>
-      <inertial>
-        <origin rpy="0 0 0" xyz="0.0092 0.00514 0"/>
-        <mass value="0.00359"/>
-        <inertia ixx= "0.00000024735"
-                 ixy= "0.00000023619"
-                 ixz= "0"
-                 iyy= "0.00000047681"
-                 iyz= "0"
-                 izz= "0.00000071813"/>
-      </inertial>
-    </link>
-    <gazebo reference="${prefix}link_median_actuating_hinge">
-      <mu1>1.1</mu1>
-      <mu2>1.1</mu2>
-    </gazebo>
-    <!-- Link median bar -->
-    <link name="${prefix}link_median_bar">
-      <visual>
-        <origin rpy="0 0 0" xyz="0.01905 0 0"/>
-        <geometry>
-          <box size="0.0381 .0075 .002"/>
-        </geometry>
-      </visual>
-      <collision>
-        <origin rpy="0 0 0" xyz="0.01905 0 0"/>
-         <geometry>
-          <box size="0.0381 .0075 .002"/>
-        </geometry>
-      </collision>
-      <inertial>
-        <origin rpy="0 0 0" xyz="0.01905 -0.00107 0"/>
-        <mass value="0.00538"/>
-        <inertia ixx= "0.00000006639"
-                 ixy="-0.00000010996"
-                 ixz= "0.00000000094"
-                 iyy= "0.00000305318"
-                 iyz= "0"
-                 izz= "0.00000304657"/>
-      </inertial>
-    </link>
-    <gazebo reference="${prefix}link_median_bar">
-      <mu1>1.1</mu1>
-      <mu2>1.1</mu2>
-    </gazebo>
-    <!-- Link paramedian hinge -->
-    <link name="${prefix}link_paramedian_hinge">
-      <visual>
-        <origin rpy="0 0 0" xyz="0 0 0"/>
-        <geometry>
-          <box size=".02 .02 .002"/>
-        </geometry>
-      </visual>
-      <collision>
-        <origin rpy="0 0 0" xyz="0 0 0"/>
-         <geometry>
-          <box size=".02 .02 .002"/>
-        </geometry>
-      </collision>
-      <inertial>
-        <origin rpy="0 0 0" xyz="-0.01025 0.00046 0"/>
-        <mass value="0.00276"/>
-        <inertia ixx= "0.00000004213"
-                 ixy="-0.00000001491"
-                 ixz= "0"
-                 iyy= "0.00000050258"
-                 iyz= "0"
-                 izz= "0.00000054007"/>
-      </inertial>
-    </link>
-    <gazebo reference="${prefix}link_paramedian_hinge">
-      <mu1>1.1</mu1>
-      <mu2>1.1</mu2>
-    </gazebo>
-    <!-- Link median bar underactuated -->
-    <link name="${prefix}link_median_bar_underactuated">
-      <visual>
-        <origin rpy="0 0 0" xyz="0.01905 0 0"/>
-        <geometry>
-          <box size="0.0381 .0075 .002"/>
-        </geometry>
-      </visual>
-      <collision>
-        <origin rpy="0 0 0" xyz="0.01905 0 0"/>
-         <geometry>
-          <box size="0.0381 .0075 .002"/>
-        </geometry>
-      </collision>
-      <inertial>
-        <origin rpy="0 0 0" xyz="0.01905 -0.00107 0"/>
-        <mass value="0.00538"/>
-        <inertia ixx= "0.00000006639"
-                 ixy="-0.00000010996"
-                 ixz="-0.00000000094"
-                 iyy= "0.00000305318"
-                 iyz= "0"
-                 izz= "0.00000304657"/>
-      </inertial>
-    </link>
-    <gazebo reference="${prefix}link_median_bar_underactuated">
-      <mu1>1.1</mu1>
-      <mu2>1.1</mu2>
-    </gazebo>
-    <!-- Link paradistal hinge -->
-    <link name="${prefix}link_paradistal_hinge">
-      <visual>
-        <origin rpy="0 0 0" xyz="0 0 0"/>
-        <geometry>
-          <box size=".02 .02 .002"/>
-        </geometry>
-      </visual>
-      <collision>
-        <origin rpy="0 0 0" xyz="0 0 0"/>
-         <geometry>
-          <box size=".02 0.02 .002"/>
-        </geometry>
-      </collision>
-      <inertial>
-        <origin rpy="0 0 0" xyz="0.00548 0 0"/>
-        <mass value="0.00158"/>
-        <inertia ixx= "0.00000001907"
-                 ixy= "0"
-                 ixz= "0"
-                 iyy= "0.00000010970"
-                 iyz= "0"
-                 izz= "0.00000012610"/>
-      </inertial>
-    </link>
-    <gazebo reference="${prefix}link_paradistal_hinge">
-      <mu1>1.1</mu1>
-      <mu2>1.1</mu2>
-    </gazebo>
-    <!-- End of link list -->
-    <!-- Joint list -->
-    <!-- Joint proximal actuating hinge -->
-    <joint name="${prefix}joint_proximal_actuating_hinge" type="revolute">
-      <parent link="${prefix}link_0"/>
-      <child link="${prefix}link_proximal_actuating_hinge"/>
-      <axis xyz="0 0 1"/>
-      <origin rpy="0 0 -2.0906" xyz="0 0 0.01"/>
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
File: robotiq_3f_gripper_visualization/cfg/robotiq_hand_with_gazebo_plugin.xacro (robot description, xacro)
@@ -1,12 +1,8 @@
 <?xml version="1.0" ?>
-<!--
-robotiq-3f-gripper_articulated - articulated version of the robotiq robotiq-3f-gripper,
-3 fingered gripper.
--->
 <robot name="robotiq-3f-gripper_articulated" xmlns:xacro="http://ros.org/wiki/xacro">
         <link name="world"/>
         <xacro:include filename="$(find robotiq_3f_gripper_visualization)/cfg/robotiq_hand_macro.urdf.xacro" />
         <xacro:robotiq_hand prefix="l_" parent="world">
-                <origin xyz="0 0 0.1" rpy="0 0 0" />
+                <origin xyz="0 0 0.1" rpy="0 1 0" />
         </xacro:robotiq_hand>
         <gazebo>
@@ -16,7 +12,3 @@
                 </plugin>
         </gazebo>
-<!--
-        <xacro:include filename="$(find robotiq_3f_gripper_visualization)/cfg/robotiq-3f-gripper_finger_articulated_macro.xacro" />
-        <xacro:robotiq-3f-gripper_finger_articulated prefix=""/>
--->
 </robot>

Commit message: tune PID & dampings for faster simulation

File: robotiq_3f_gripper_visualization/cfg/robotiq_hand_macro.urdf.xacro (robot description, xacro)
@@ -601,5 +601,5 @@
             <parent link="${prefix}link_0"/>
             <child link="${prefix}link_1"/>
-            <dynamics damping="1" friction="0"/>
+            <dynamics damping="0.1" friction="0"/>
             <!-- Limits: [0deg.,70deg.] -->
             <limit effort="60" velocity="-1" lower="0" upper="1.2217"/>
@@ -612,5 +612,5 @@
             <parent link="${prefix}link_1"/>
             <child link="${prefix}link_2"/>
-            <dynamics damping="1" friction="0"/>
+            <dynamics damping="0.1" friction="0"/>
             <axis xyz="0 0 1"/>
             <origin rpy="0 0 0" xyz="0 0.05715 0"/>
@@ -625,5 +625,5 @@
             <parent link="${prefix}link_2"/>
             <child link="${prefix}link_3"/>
-            <dynamics damping="1" friction="0"/>
+            <dynamics damping="0.1" friction="0"/>
             <axis xyz="0 0 1"/>
             <origin rpy="0 0 ${3.1416/2 + 0.5198}" xyz="0 0.039 0"/>
@@ -782,5 +782,5 @@
             <parent link="${prefix}palm"/>
             <child link="${prefix}finger_1_link_0"/>
-            <dynamics damping="1" friction="0"/>
+            <dynamics damping="0.1" friction="0"/>
             <axis xyz="0 1 0"/>
             <origin rpy="0 3.1416 -1.57" xyz="-0.0455 0.0214 0.036"/>
@@ -795,5 +795,5 @@
             <parent link="${prefix}palm"/>
             <child link="${prefix}finger_2_link_0"/>
-            <dynamics damping="1" friction="0"/>
+            <dynamics damping="0.1" friction="0"/>
             <axis xyz="0 1 0"/>
             <origin rpy="0 3.1416 -1.57" xyz="-0.0455 0.0214 -0.036"/>
@@ -808,5 +808,5 @@
             <parent link="${prefix}palm"/>
             <child link="${prefix}finger_middle_link_0"/>
-            <dynamics damping="1" friction="0"/>
+            <dynamics damping="0.1" friction="0"/>
             <axis xyz="0 1 0"/>
             <origin rpy="0 0 1.57" xyz="0.0455 0.0214 0"/>

File: robotiq_3f_gripper_visualization/cfg/robotiq_hand_with_gazebo_plugin.xacro (robot description, xacro)
@@ -1,14 +1,15 @@
 <?xml version="1.0" ?>
 <robot name="robotiq-3f-gripper_articulated" xmlns:xacro="http://ros.org/wiki/xacro">
-        <link name="world"/>
-        <xacro:include filename="$(find robotiq_3f_gripper_visualization)/cfg/robotiq_hand_macro.urdf.xacro" />
-        <xacro:robotiq_hand prefix="l_" parent="world">
-                <origin xyz="0 0 0.1" rpy="0 1 0" />
-        </xacro:robotiq_hand>
-        <gazebo>
-                <plugin name="RobotiqHandPlugin" filename="libRobotiqHandPlugin.so">
-                        <side>left</side>
-                        <kp_position>5</kp_position>
-                </plugin>
-        </gazebo>
+    <link name="world"/>
+    <xacro:include filename="$(find robotiq_3f_gripper_visualization)/cfg/robotiq_hand_macro.urdf.xacro"/>
+    <xacro:robotiq_hand prefix="l_" parent="world">
+        <origin xyz="0 0 0.1" rpy="0 1 0"/>
+    </xacro:robotiq_hand>
+    <gazebo>
+        <plugin name="RobotiqHandPlugin" filename="libRobotiqHandPlugin.so">
+            <side>left</side>
+            <kp_position>0.2</kp_position>
+            <kd_position>0.05</kd_position>
+        </plugin>
+    </gazebo>
 </robot>

Commit message: two types of grippers
one kinematic which is faster and more stable to simulate
the other is not kinematic, which can be used to simulate actual grasping

File: robotiq_3f_gripper_visualization/cfg/robotiq_hand_macro.urdf.xacro (robot description, xacro)
@@ -7,5 +7,5 @@
 -->
 <robot xmlns:xacro="http://www.ros.org/wiki/xacro" name="robotiq_hand">
-    <xacro:macro name="robotiq_finger" params="prefix">
+    <xacro:macro name="robotiq_finger" params="prefix kinematic">
         <!-- Link list -->
         <!-- Link 0 -->
@@ -36,4 +36,5 @@
         </link>
         <gazebo reference="${prefix}link_0">
+            <kinematic>${kinematic}</kinematic>
             <mu1>1.1</mu1>
             <mu2>1.1</mu2>
@@ -76,4 +77,5 @@
         </link>
         <gazebo reference="${prefix}link_1">
+            <kinematic>${kinematic}</kinematic>
             <mu1>1.1</mu1>
             <mu2>1.1</mu2>
@@ -114,4 +116,5 @@
         </link>
         <gazebo reference="${prefix}link_2">
+            <kinematic>${kinematic}</kinematic>
             <mu1>1.1</mu1>
             <mu2>1.1</mu2>
@@ -152,4 +155,5 @@
         </link>
         <gazebo reference="${prefix}link_3">
+            <kinematic>${kinematic}</kinematic>
             <mu1>1.1</mu1>
             <mu2>1.1</mu2>
@@ -188,4 +192,5 @@
         </link>
         <gazebo reference="${prefix}link_proximal_actuating_hinge">
+            <kinematic>${kinematic}</kinematic>
             <mu1>1.1</mu1>
             <mu2>1.1</mu2>
@@ -225,4 +230,5 @@
         </link>
         <gazebo reference="${prefix}link_paraproximal_actuating_hinge">
+            <kinematic>${kinematic}</kinematic>
             <mu1>1.1</mu1>
             <mu2>1.1</mu2>
@@ -261,4 +267,5 @@
         </link>
         <gazebo reference="${prefix}link_proximal_actuating_bar">
+            <kinematic>${kinematic}</kinematic>
             <mu1>1.1</mu1>
             <mu2>1.1</mu2>
@@ -297,4 +304,5 @@
         </link>
         <gazebo reference="${prefix}link_paraproximal_bar">
+            <kinematic>${kinematic}</kinematic>
             <mu1>1.1</mu1>
             <mu2>1.1</mu2>
@@ -333,4 +341,5 @@
         </link>
         <gazebo reference="${prefix}link_median_actuating_hinge">
+            <kinematic>${kinematic}</kinematic>
             <mu1>1.1</mu1>
             <mu2>1.1</mu2>
@@ -369,4 +378,5 @@
         </link>
         <gazebo reference="${prefix}link_median_bar">
+            <kinematic>${kinematic}</kinematic>
             <mu1>1.1</mu1>
             <mu2>1.1</mu2>
@@ -405,4 +415,5 @@
         </link>
         <gazebo reference="${prefix}link_paramedian_hinge">
+            <kinematic>${kinematic}</kinematic>
             <mu1>1.1</mu1>
             <mu2>1.1</mu2>
@@ -441,4 +452,5 @@
         </link>
         <gazebo reference="${prefix}link_median_bar_underactuated">
+            <kinematic>${kinematic}</kinematic>
             <mu1>1.1</mu1>
             <mu2>1.1</mu2>
@@ -477,4 +489,5 @@
         </link>
         <gazebo reference="${prefix}link_paradistal_hinge">
+            <kinematic>${kinematic}</kinematic>
             <mu1>1.1</mu1>
             <mu2>1.1</mu2>
@@ -727,5 +740,5 @@
         </gazebo>
     </xacro:macro>
-    <xacro:macro name="robotiq_hand" params="prefix *origin parent">
+    <xacro:macro name="robotiq_hand" params="prefix *origin parent kinematic">
         <!-- joint attaching parent link to robotiq hand -->
         <joint name="${prefix}robotiq_hand_joint" type="fixed">
@@ -735,7 +748,7 @@
         </joint>
         <!-- Insert the fingers -->
-        <xacro:robotiq_finger prefix="${prefix}finger_1_"/>
-        <xacro:robotiq_finger prefix="${prefix}finger_2_"/>
-        <xacro:robotiq_finger prefix="${prefix}finger_middle_"/>
+        <xacro:robotiq_finger prefix="${prefix}finger_1_" kinematic="${kinematic}"/>
+        <xacro:robotiq_finger prefix="${prefix}finger_2_" kinematic="${kinematic}"/>
+        <xacro:robotiq_finger prefix="${prefix}finger_middle_" kinematic="${kinematic}"/>
         <!-- link list -->
         <!-- Link palm -->
@@ -766,4 +779,5 @@
         </link>
         <gazebo reference="${prefix}palm">
+            <kinematic>${kinematic}</kinematic>
             <mu1>1.1</mu1>
             <mu2>1.1</mu2>
