Commit message: make the knuckle joint of the middle finger fixed

File: robotiq_3f_gripper_visualization/cfg/kinematic_robotiq_hand_macro.urdf.xacro (robot description, xacro)
@@ -283,5 +283,5 @@
         </gazebo>
         <!-- Joint palm_finger_middle_joint -->
-        <joint name="${prefix}palm_finger_middle_joint" type="revolute">
+        <joint name="${prefix}palm_finger_middle_joint" type="fixed">
             <parent link="${prefix}palm"/>
             <child link="${prefix}finger_middle_link_0"/>
